Commit message: added second Hokuyo scanner to the back of the base because this is the most common setup now, for simulation noise was added to the laser scanners, and because of some movement issues in gazebo joint control was switched to PositionJointInterface

File: robots/youbot.urdf.xacro (robot description, xacro)
@@ -42,6 +42,10 @@
   </xacro:youbot_gripper>
   <!-- base laser front -->
-  <xacro:hokuyo_urg04_laser name="base_laser_front" parent="base" ros_topic="scan_front" update_rate="10" min_angle="-1.57" max_angle="1.57">
+  <xacro:hokuyo_urg04_laser name="base_laser_front" parent="base" ros_topic="base_scan" update_rate="10" min_angle="-1.57" max_angle="1.57">
     <origin xyz="0.3 0 -0.03" rpy="0 0 0"/>
   </xacro:hokuyo_urg04_laser>
+  <!-- base laser back -->
+  <xacro:hokuyo_urg04_laser name="base_laser_back" parent="base" ros_topic="base_scan_back" update_rate="10" min_angle="-1.57" max_angle="1.57">
+    <origin xyz="-0.3 0 -0.03" rpy="0 0 ${M_PI}"/>
+  </xacro:hokuyo_urg04_laser>
 </robot>

File: urdf/youbot_arm/arm.transmission.xacro (robot description, xacro)
@@ -4,57 +4,57 @@
        xmlns:interface="http://playerstage.sourceforge.net/gazebo/xmlschema/#interface"
        xmlns:xacro="http://ros.org/wiki/xacro">
-  <!-- reduction ratio doesn't affect the model-->
-  <!-- reduction ratio must not to be 0-->
-  <xacro:macro name="youbot_arm_transmission" params="name">
-    <transmission name="${name}_trans_1">
+	<!-- reduction ratio doesn't affect the model-->
+	<!-- reduction ratio must not to be 0-->
+	<xacro:macro name="youbot_arm_transmission" params="name">
+		<transmission name="${name}_trans_1">
       <type>transmission_interface/SimpleTransmission</type>
-      <actuator name="${name}_motor_1">
-        <hardwareInterface>EffortJointInterface</hardwareInterface>
+			<actuator name="${name}_motor_1">
+        <hardwareInterface>PositionJointInterface</hardwareInterface>
         <mechanicalReduction>1</mechanicalReduction>
       </actuator>
-      <joint name="${name}_joint_1">
-        <hardwareInterface>EffortJointInterface</hardwareInterface>
+			<joint name="${name}_joint_1">
+        <hardwareInterface>PositionJointInterface</hardwareInterface>
       </joint>
-    </transmission>
-    <transmission name="${name}_trans_2">
+		</transmission>
+		<transmission name="${name}_trans_2">
       <type>transmission_interface/SimpleTransmission</type>
-      <actuator name="${name}_motor_2">
-        <hardwareInterface>EffortJointInterface</hardwareInterface>
+			<actuator name="${name}_motor_2">
+        <hardwareInterface>PositionJointInterface</hardwareInterface>
         <mechanicalReduction>1</mechanicalReduction>
       </actuator>
-      <joint name="${name}_joint_2">
-        <hardwareInterface>EffortJointInterface</hardwareInterface>
+			<joint name="${name}_joint_2">
+        <hardwareInterface>PositionJointInterface</hardwareInterface>
       </joint>
-    </transmission>
-    <transmission name="${name}_trans_3">
+		</transmission>
+		<transmission name="${name}_trans_3">
       <type>transmission_interface/SimpleTransmission</type>
-      <actuator name="${name}_motor_3">
-        <hardwareInterface>EffortJointInterface</hardwareInterface>
+			<actuator name="${name}_motor_3">
+        <hardwareInterface>PositionJointInterface</hardwareInterface>
         <mechanicalReduction>1</mechanicalReduction>
       </actuator>
-      <joint name="${name}_joint_3">
-        <hardwareInterface>EffortJointInterface</hardwareInterface>
+			<joint name="${name}_joint_3">
+        <hardwareInterface>PositionJointInterface</hardwareInterface>
       </joint>
-    </transmission>
-    <transmission name="${name}_trans_4">
+		</transmission>
+		<transmission name="${name}_trans_4">
       <type>transmission_interface/SimpleTransmission</type>
-      <actuator name="${name}_motor_4">
-        <hardwareInterface>EffortJointInterface</hardwareInterface>
+			<actuator name="${name}_motor_4">
+        <hardwareInterface>PositionJointInterface</hardwareInterface>
         <mechanicalReduction>1</mechanicalReduction>
       </actuator>
-      <joint name="${name}_joint_4">
-        <hardwareInterface>EffortJointInterface</hardwareInterface>
+			<joint name="${name}_joint_4">
+        <hardwareInterface>PositionJointInterface</hardwareInterface>
       </joint>
-    </transmission>
-    <transmission name="${name}_trans_5">
+		</transmission>
+		<transmission name="${name}_trans_5">
       <type>transmission_interface/SimpleTransmission</type>
-      <actuator name="${name}_motor_5">
-        <hardwareInterface>EffortJointInterface</hardwareInterface>
+			<actuator name="${name}_motor_5">
+        <hardwareInterface>PositionJointInterface</hardwareInterface>
         <mechanicalReduction>1</mechanicalReduction>
       </actuator>
-      <joint name="${name}_joint_5">
-        <hardwareInterface>EffortJointInterface</hardwareInterface>
+			<joint name="${name}_joint_5">
+        <hardwareInterface>PositionJointInterface</hardwareInterface>
       </joint>
-    </transmission>
-  </xacro:macro>
+		</transmission>
+	</xacro:macro>
 </robot>

File: urdf/youbot_gripper/gripper.transmission.xacro (robot description, xacro)
@@ -4,25 +4,25 @@
        xmlns:interface="http://playerstage.sourceforge.net/gazebo/xmlschema/#interface"
        xmlns:xacro="http://ros.org/wiki/xacro">
-  <xacro:macro name="youbot_gripper_transmission" params="name">
-    <transmission name="${name}_finger_l_trans">
+	<xacro:macro name="youbot_gripper_transmission" params="name">
+		<transmission name="${name}_finger_l_trans">
       <type>transmission_interface/SimpleTransmission</type>
-      <actuator name="${name}_finger_l_motor">
-        <hardwareInterface>EffortJointInterface</hardwareInterface>
+			<actuator name="${name}_finger_l_motor">
+        <hardwareInterface>PositionJointInterface</hardwareInterface>
         <mechanicalReduction>1</mechanicalReduction>
       </actuator>
-      <joint name="${name}_finger_joint_l">
-        <hardwareInterface>EffortJointInterface</hardwareInterface>
+			<joint name="${name}_finger_joint_l">
+        <hardwareInterface>PositionJointInterface</hardwareInterface>
       </joint>
-    </transmission>
-    <transmission name="${name}_finger_r_trans">
+		</transmission>
+		<transmission name="${name}_finger_r_trans">
       <type>transmission_interface/SimpleTransmission</type>
-      <actuator name="${name}_finger_r_motor">
-        <hardwareInterface>EffortJointInterface</hardwareInterface>
+			<actuator name="${name}_finger_r_motor">
+        <hardwareInterface>PositionJointInterface</hardwareInterface>
         <mechanicalReduction>1</mechanicalReduction>
       </actuator>
-      <joint name="${name}_finger_joint_r">
-        <hardwareInterface>EffortJointInterface</hardwareInterface>
+			<joint name="${name}_finger_joint_r">
+        <hardwareInterface>PositionJointInterface</hardwareInterface>
       </joint>
-    </transmission>
-  </xacro:macro>
+		</transmission>
+	</xacro:macro>
 </robot>
