Commit message: added gaussian noise to laser scanner

File: urdf/sensors/hokuyo_urg04_laser.gazebo.xacro (robot description, xacro)
@@ -1,38 +1,44 @@
 <?xml version="1.0"?>
 <robot xmlns:sensor="http://playerstage.sourceforge.net/gazebo/xmlschema/#sensor"
-       xmlns:controller="http://playerstage.sourceforge.net/gazebo/xmlschema/#controller"
-       xmlns:interface="http://playerstage.sourceforge.net/gazebo/xmlschema/#interface"
-       xmlns:xacro="http://ros.org/wiki/xacro">
-  <xacro:macro name="hokuyo_urg04_laser_gazebo" params="name ros_topic update_rate min_angle max_angle">
-    <gazebo reference="${name}_link">
-      <sensor name="${name}" type="ray">
-		<always_on>true</always_on>
-        <update_rate>${update_rate}</update_rate>
-		<pose>0 0 0 0 0 0</pose>
-		<visualize>false</visualize>
-        <ray>
-            <scan>
-                <horizontal>
-                    <samples>150</samples>
-                    <resolution>1.0</resolution>
-                    <min_angle>${min_angle}</min_angle>
-                    <max_angle>${max_angle}</max_angle>
-                </horizontal>
-            </scan>
-            <range>
-				<min>0.05</min>
-				<max>5.6</max>
-				<resolution>0.36</resolution>
-			</range>
-        </ray>
-        <plugin name="gazebo_ros_${name}_controller" filename="libgazebo_ros_laser.so">
-            <gaussianNoise>0.005</gaussianNoise>
-            <alwaysOn>true</alwaysOn>
-            <updateRate>${update_rate}</updateRate>
-            <topicName>${ros_topic}</topicName>
-            <frameName>/${name}_link</frameName>
-         </plugin>
-      </sensor>
-    </gazebo>
-  </xacro:macro>
+	xmlns:controller="http://playerstage.sourceforge.net/gazebo/xmlschema/#controller"
+	xmlns:interface="http://playerstage.sourceforge.net/gazebo/xmlschema/#interface"
+	xmlns:xacro="http://ros.org/wiki/xacro">
+	<xacro:macro name="hokuyo_urg04_laser_gazebo"
+		params="name ros_topic update_rate min_angle max_angle">
+		<gazebo reference="${name}_link">
+			<sensor name="${name}" type="ray">
+				<always_on>true</always_on>
+				<update_rate>${update_rate}</update_rate>
+				<pose>0 0 0 0 0 0</pose>
+				<visualize>false</visualize>
+				<ray>
+					<scan>
+						<horizontal>
+							<samples>150</samples>
+							<resolution>1.0</resolution>
+							<min_angle>${min_angle}</min_angle>
+							<max_angle>${max_angle}</max_angle>
+						</horizontal>
+					</scan>
+					<range>
+						<min>0.05</min>
+						<max>5.6</max>
+						<resolution>0.36</resolution>
+					</range>
+					<noise>
+						<type>gaussian</type>
+						<mean>0.0</mean>
+						<stddev>0.01</stddev>
+					</noise>
+				</ray>
+				<plugin name="gazebo_ros_${name}_controller" filename="libgazebo_ros_laser.so">
+					<gaussianNoise>0.005</gaussianNoise>
+					<alwaysOn>true</alwaysOn>
+					<updateRate>${update_rate}</updateRate>
+					<topicName>${ros_topic}</topicName>
+					<frameName>/${name}_link</frameName>
+				</plugin>
+			</sensor>
+		</gazebo>
+	</xacro:macro>
 </robot>
