Commit message: migrated files to Jade

File: controller/ros_controller.urdf.xacro (robot description, xacro)
@@ -2,5 +2,6 @@
 <robot xmlns:sensor="http://playerstage.sourceforge.net/gazebo/xmlschema/#sensor"
        xmlns:controller="http://playerstage.sourceforge.net/gazebo/xmlschema/#controller"
-       xmlns:interface="http://playerstage.sourceforge.net/gazebo/xmlschema/#interface">
+       xmlns:interface="http://playerstage.sourceforge.net/gazebo/xmlschema/#interface"
+       xmlns:xacro="http://ros.org/wiki/xacro">
   <gazebo>
     <plugin name="gazebo_ros_controller" filename="libgazebo_ros_control.so" />

File: robots/youbot.urdf.xacro (robot description, xacro)
@@ -3,5 +3,5 @@
        xmlns:controller="http://playerstage.sourceforge.net/gazebo/xmlschema/#controller"
        xmlns:interface="http://playerstage.sourceforge.net/gazebo/xmlschema/#interface"
-       xmlns:xacro="http://playerstage.sourceforge.net/gazebo/xmlschema/#interface"
+       xmlns:xacro="http://ros.org/wiki/xacro"
        name="youbot" >
   <!-- The following xacro:included files set up definitions of parts of the robot body -->

File: robots/youbot_base_only.urdf.xacro (robot description, xacro)
@@ -3,5 +3,5 @@
        xmlns:controller="http://playerstage.sourceforge.net/gazebo/xmlschema/#controller"
        xmlns:interface="http://playerstage.sourceforge.net/gazebo/xmlschema/#interface"
-       xmlns:xacro="http://playerstage.sourceforge.net/gazebo/xmlschema/#interface"
+       xmlns:xacro="http://ros.org/wiki/xacro"
        name="youbot" >
   <!-- The following xacro:included files set up definitions of parts of the robot body -->

File: robots/youbot_dual_arm.urdf.xacro (robot description, xacro)
@@ -3,5 +3,5 @@
        xmlns:controller="http://playerstage.sourceforge.net/gazebo/xmlschema/#controller"
        xmlns:interface="http://playerstage.sourceforge.net/gazebo/xmlschema/#interface"
-       xmlns:xacro="http://playerstage.sourceforge.net/gazebo/xmlschema/#interface"
+       xmlns:xacro="http://ros.org/wiki/xacro"
        name="youbot" >
   <!-- The following xacro:included files set up definitions of parts of the robot body -->

File: robots/youbot_with_cam3d.urdf.xacro (robot description, xacro)
@@ -3,5 +3,5 @@
        xmlns:controller="http://playerstage.sourceforge.net/gazebo/xmlschema/#controller"
        xmlns:interface="http://playerstage.sourceforge.net/gazebo/xmlschema/#interface"
-       xmlns:xacro="http://playerstage.sourceforge.net/gazebo/xmlschema/#interface"
+       xmlns:xacro="http://ros.org/wiki/xacro"
        name="youbot" >
   <!-- The following xacro:included files set up definitions of parts of the robot body -->

File: urdf/materials.urdf.xacro (robot description, xacro)
@@ -1,4 +1,4 @@
 <?xml version="1.0"?>
-<robot>
+<robot xmlns:xacro="http://ros.org/wiki/xacro">
   <material name="youBot/Orange">
     <color rgba="1.0 0.4 0.0 1.0"/>

File: urdf/misc/camera_tower.urdf.xacro (robot description, xacro)
@@ -4,7 +4,7 @@
        xmlns:interface="http://playerstage.sourceforge.net/gazebo/xmlschema/#interface"
        xmlns:xacro="http://ros.org/wiki/xacro">
-  <property name="camera_tower_height" value="0.49" />
-  <property name="camera_tower_width" value="0.03" />
-  <property name="camera_tower_depth" value="0.03" />
+  <xacro:property name="camera_tower_height" value="0.49" />
+  <xacro:property name="camera_tower_width" value="0.03" />
+  <xacro:property name="camera_tower_depth" value="0.03" />
   <xacro:macro name="camera_tower" params="name parent *origin">
   	<link name="${name}_link">
@@ -29,5 +29,5 @@
     </link>
     <joint name="${name}_joint" type="fixed">
-      <insert_block name="origin" />
+      <xacro:insert_block name="origin" />
       <parent link="${parent}"/>
       <child link="${name}_link"/>

File: urdf/sensors/asus_xtion_camera.urdf.xacro (robot description, xacro)
@@ -1,7 +1,7 @@
 <?xml version="1.0"?>
-<root xmlns:xacro="http://playerstage.sourceforge.net/gazebo/xmlschema/#interface">
+<root xmlns:xacro="http://ros.org/wiki/xacro">
   <xacro:include filename="$(find youbot_description)/urdf/sensors/asus_xtion_camera.gazebo.xacro" />
-  <property name="eye_x_offset" value="0.03" />
-  <property name="eye_y_offset" value="0.035" />
+  <xacro:property name="eye_x_offset" value="0.03" />
+  <xacro:property name="eye_y_offset" value="0.035" />
   <xacro:macro name="asus_xtion_eye" params="suffix parent *origin">
 	<link name="${parent}_${suffix}_frame">
@@ -15,5 +15,5 @@
 	  <parent link="${parent}_camera"/>
 	  <child link="${parent}_${suffix}_frame"/>
-	  <insert_block name="origin"/>
+	  <xacro:insert_block name="origin"/>
 	</joint>
   </xacro:macro>
@@ -40,5 +40,5 @@
     </link>
     <joint name="${name}_foot_joint" type="fixed">
-      <insert_block name="origin" />
+      <xacro:insert_block name="origin" />
       <parent link="${parent}"/>
       <child link="${name}_foot_link"/>

File: urdf/youbot_arm/arm.urdf.xacro (robot description, xacro)
@@ -10,5 +10,5 @@
 		<!-- joint between base_link and arm_0_link -->
 		<joint name="${name}_joint_0" type="fixed" >
-			<insert_block name="origin" />
+			<xacro:insert_block name="origin" />
 			<parent link="${parent}" />
 			<child link="${name}_link_0" />

File: urdf/youbot_arm/limits.urdf.xacro (robot description, xacro)
@@ -1,31 +1,31 @@
 <?xml version="1.0"?>
-<robot xmlns:xacro="http://ros.org/wiki/xacro">>
+<robot xmlns:xacro="http://ros.org/wiki/xacro">
 	<!-- common properties -->
-	<property name="M_PI" value="3.1415926535897931" />
-	<property name="threshold" value="0.01" />
+	<xacro:property name="M_PI" value="3.1415926535897931" />
+	<xacro:property name="threshold" value="0.01" />
 	<!-- arm limits positions (deg) -->
-	<property name="joint_1_limit" value="${M_PI * (169 + 169) / 180}" />
-	<property name="joint_2_limit" value="${M_PI * (90 + 65) / 180}" />
-	<property name="joint_3_limit" value="${M_PI * (146 + 151) / 180}" />
-	<property name="joint_4_limit" value="${M_PI * (102.5 + 102.5) / 180}" />
-	<property name="joint_5_limit" value="${M_PI * (167.5 + 167.5) / 180}" />
-	<property name="joint_1_limit_soft" value="${joint_1_limit - threshold}" />
-	<property name="joint_2_limit_soft" value="${joint_2_limit - threshold}" />
-	<property name="joint_3_limit_soft" value="${joint_3_limit - threshold}" />
-	<property name="joint_4_limit_soft" value="${joint_4_limit - threshold}" />
-	<property name="joint_5_limit_soft" value="${joint_5_limit - threshold}" />
+	<xacro:property name="joint_1_limit" value="${M_PI * (169 + 169) / 180}" />
+	<xacro:property name="joint_2_limit" value="${M_PI * (90 + 65) / 180}" />
+	<xacro:property name="joint_3_limit" value="${M_PI * (146 + 151) / 180}" />
+	<xacro:property name="joint_4_limit" value="${M_PI * (102.5 + 102.5) / 180}" />
+	<xacro:property name="joint_5_limit" value="${M_PI * (167.5 + 167.5) / 180}" />
+	<xacro:property name="joint_1_limit_soft" value="${joint_1_limit - threshold}" />
+	<xacro:property name="joint_2_limit_soft" value="${joint_2_limit - threshold}" />
+	<xacro:property name="joint_3_limit_soft" value="${joint_3_limit - threshold}" />
+	<xacro:property name="joint_4_limit_soft" value="${joint_4_limit - threshold}" />
+	<xacro:property name="joint_5_limit_soft" value="${joint_5_limit - threshold}" />
 	<!-- dynamic properties : mass (kg) Alu data sheet -->
-	<property name="link_0_mass" value="0.961" />
-	<property name="link_1_mass" value="1.390" />
-	<property name="link_2_mass" value="1.318" />
-	<property name="link_3_mass" value="0.821" />
-	<property name="link_4_mass" value="0.769" />
-	<property name="link_5_mass" value="0.687" />
-	<!--<property name="link_0_mass" value="0.845" />
-	<property name="link_1_mass" value="0.1" />
-	<property name="link_2_mass" value="0.1" />
-	<property name="link_3_mass" value="0.1" />
-	<property name="link_4_mass" value="0.1" />
-	<property name="link_5_mass" value="0.1" />-->
+	<xacro:property name="link_0_mass" value="0.961" />
+	<xacro:property name="link_1_mass" value="1.390" />
+	<xacro:property name="link_2_mass" value="1.318" />
+	<xacro:property name="link_3_mass" value="0.821" />
+	<xacro:property name="link_4_mass" value="0.769" />
+	<xacro:property name="link_5_mass" value="0.687" />
+	<!--<xacro:property name="link_0_mass" value="0.845" />
+	<xacro:property name="link_1_mass" value="0.1" />
+	<xacro:property name="link_2_mass" value="0.1" />
+	<xacro:property name="link_3_mass" value="0.1" />
+	<xacro:property name="link_4_mass" value="0.1" />
+	<xacro:property name="link_5_mass" value="0.1" />-->
 	<!-- TODO: add inertia tensor-->
 	<xacro:macro name="default_origin">

File: urdf/youbot_base/base.transmission.xacro (robot description, xacro)
@@ -4,7 +4,6 @@
        xmlns:interface="http://playerstage.sourceforge.net/gazebo/xmlschema/#interface"
        xmlns:xacro="http://ros.org/wiki/xacro">
-  <property name="wheel_mechanical_reduction" value="${624/35 * 80/18}" />
-  <property name="caster_mechanical_reduction" value="${624/35 * 80/18}" />
-  <property name="" value="0.360" />
+  <xacro:property name="wheel_mechanical_reduction" value="${624/35 * 80/18}" />
+  <xacro:property name="caster_mechanical_reduction" value="${624/35 * 80/18}" />
   <xacro:macro name="youbot_base_transmission">
   <!-- front left wheel -->

File: urdf/youbot_base/base.urdf.xacro (robot description, xacro)
@@ -7,28 +7,28 @@
   <xacro:include filename="$(find youbot_description)/urdf/youbot_base/base.transmission.xacro"/>
   <!-- simplified box collision geometry for base -->
-  <property name="base_size_x" value="0.570"/>
-  <property name="base_size_y" value="0.360"/>
-  <property name="base_size_z" value="0.100"/>
-  <property name="base_mass" value="22.0"/>
-  <property name="caster_offset_x" value="0.228"/>
-  <property name="caster_offset_y" value="0.158"/>
-  <property name="caster_offset_z" value="-0.034"/>
-  <property name="caster_mass" value="0.1"/>
-  <property name="wheel_offset_x" value="0.0"/>
-  <property name="wheel_offset_y" value="0.0"/>
-  <property name="wheel_offset_z" value="0.0"/>
-  <property name="wheel_mass" value="1.4"/>
-  <property name="wheel_radius" value="0.0475"/>
-  <property name="wheel_length" value="0.005"/>
-  <property name="caster_joint_damping" value="1.0"/>
-  <property name="caster_joint_friction" value="1.0"/>
-  <property name="caster_joint_effort" value="30"/>
-  <property name="caster_joint_velocity" value="10"/>
-  <property name="caster_joint_safety_k_velocity" value="10.0"/>
-  <property name="wheel_joint_damping" value="1.0"/>
-  <property name="wheel_joint_friction" value="1.0"/>
-  <property name="wheel_joint_effort" value="30"/>
-  <property name="wheel_joint_velocity" value="10"/>
-  <property name="wheel_joint_safety_k_velocity" value="10.0"/>
+  <xacro:property name="base_size_x" value="0.570"/>
+  <xacro:property name="base_size_y" value="0.360"/>
+  <xacro:property name="base_size_z" value="0.100"/>
+  <xacro:property name="base_mass" value="22.0"/>
+  <xacro:property name="caster_offset_x" value="0.228"/>
+  <xacro:property name="caster_offset_y" value="0.158"/>
+  <xacro:property name="caster_offset_z" value="-0.034"/>
+  <xacro:property name="caster_mass" value="0.1"/>
+  <xacro:property name="wheel_offset_x" value="0.0"/>
+  <xacro:property name="wheel_offset_y" value="0.0"/>
+  <xacro:property name="wheel_offset_z" value="0.0"/>
+  <xacro:property name="wheel_mass" value="1.4"/>
+  <xacro:property name="wheel_radius" value="0.0475"/>
+  <xacro:property name="wheel_length" value="0.005"/>
+  <xacro:property name="caster_joint_damping" value="1.0"/>
+  <xacro:property name="caster_joint_friction" value="1.0"/>
+  <xacro:property name="caster_joint_effort" value="30"/>
+  <xacro:property name="caster_joint_velocity" value="10"/>
+  <xacro:property name="caster_joint_safety_k_velocity" value="10.0"/>
+  <xacro:property name="wheel_joint_damping" value="1.0"/>
+  <xacro:property name="wheel_joint_friction" value="1.0"/>
+  <xacro:property name="wheel_joint_effort" value="30"/>
+  <xacro:property name="wheel_joint_velocity" value="10"/>
+  <xacro:property name="wheel_joint_safety_k_velocity" value="10.0"/>
   <xacro:macro name="youbot_base" params="name">
     <link name="${name}_footprint">

File: urdf/youbot_gripper/limits.urdf.xacro (robot description, xacro)
@@ -1,9 +1,9 @@
 <?xml version="1.0"?>
-<robot>
+<robot xmlns:xacro="http://ros.org/wiki/xacro">
 	<!-- common properties -->
-	<property name="M_PI" value="3.1415926535897931" />
-        <property name="threshold" value="0.001" />
+	<xacro:property name="M_PI" value="3.1415926535897931" />
+        <xacro:property name="threshold" value="0.001" />
 	<!-- fingers limits, values are in meters -->
-	<property name="finger_joint" value="${0.023 / 2.0}" />
-	<property name="finger_joint_soft" value="${(0.023 - threshold) / 2.0}" />
+	<xacro:property name="finger_joint" value="${0.023 / 2.0}" />
+	<xacro:property name="finger_joint_soft" value="${(0.023 - threshold) / 2.0}" />
 </robot>

File: urdf/youbot_plate/plate.urdf.xacro (robot description, xacro)
@@ -7,5 +7,5 @@
 		<!-- joint between arm_7_link and sdh_palm_link -->
 		<joint name="${name}_joint" type="fixed" >
-			<insert_block name="origin" />
+			<xacro:insert_block name="origin" />
 			<parent link="${parent}" />
 			<child link="${name}_link" />
